Commit message: 1.modify example 2.update configuration

File: cuarm_configuration/dual_v2_2/share/no_gripper/dual_arm.urdf (robot description, URDF)
Before this commit: robot dual_v2_2, 24 links, 23 joints
Links:
- removed link DP
- removed link s1
- removed link s2
- removed link s3
- removed link s4
- added link H1, mass 0.416514798250936; collision mesh filename=package://cuarm_mesh/dual_v2_2/meshes/base/H1.STL; visual mesh filename=package://cuarm_mesh/dual_v2_2/meshes/base/H1.STL
- added link H2, mass 0.2515794715362; collision mesh filename=package://cuarm_mesh/dual_v2_2/meshes/base/H2.STL; visual mesh filename=package://cuarm_mesh/dual_v2_2/meshes/base/H2.STL
- added link S0, mass 68.8751085446278; collision mesh filename=package://cuarm_mesh/dual_v2_2/meshes/base/S0.STL; visual mesh filename=package://cuarm_mesh/dual_v2_2/meshes/base/S0.STL
- added link S1, mass 8.59759690292358; collision mesh filename=package://cuarm_mesh/dual_v2_2/meshes/base/S1.STL; visual mesh filename=package://cuarm_mesh/dual_v2_2/meshes/base/S1.STL
- added link S2, mass 5.22090662821691; collision mesh filename=package://cuarm_mesh/dual_v2_2/meshes/base/S2.STL; visual mesh filename=package://cuarm_mesh/dual_v2_2/meshes/base/S2.STL
- added link S3, mass 4.78694804166376; collision mesh filename=package://cuarm_mesh/dual_v2_2/meshes/base/S3.STL; visual mesh filename=package://cuarm_mesh/dual_v2_2/meshes/base/S3.STL
- added link S4, mass 12.776; collision mesh filename=package://cuarm_mesh/dual_v2_2/meshes/base/S4.STL; visual mesh filename=package://cuarm_mesh/dual_v2_2/meshes/base/S4.STL
- link arm_L1_l: mass 1.8018 -> 1.7675
- link arm_L1_r: mass 1.8018 -> 1.7675
- link arm_L2_l: mass 0.72275 -> 0.38586
- link arm_L2_r: mass 0.72275 -> 0.38586
- link arm_L3_l: mass 1.7397 -> 1.7244
- link arm_L3_r: mass 1.7397 -> 1.7244
- link arm_L4_l: mass 1.299 -> 1.371
- link arm_L4_r: mass 1.299 -> 1.371
- link arm_L5_l: mass 0.94391 -> 1.0029
- link arm_L5_r: mass 0.94391 -> 1.0029
- link arm_L6_l: mass 0.87461 -> 0.831539795358367
- link arm_L6_r: mass 0.87461 -> 0.83154
- link arm_L7_l: mass 0.75543 -> 0.45531
- link arm_L7_r: mass 0.75543 -> 0.45531
Joints:
- removed joint s1j
- removed joint s2j
- removed joint s3j
- removed joint s4j
- added joint H1j: type revolute, parent S4, child H1, origin xyz= -0.0215      0.000000000  0.5581      rpy= 0.000000000  0.000000000  0.000000000, axis 0 0 1, limit lower=0 upper=0 effort=0 velocity=0
- added joint H2j: type revolute, parent H1, child H2, origin xyz= 0.000000000  0.000000000  0.000000000 rpy= -1.5708      0.000000000  0.000000000, axis 0 0 1, limit lower=0 upper=0 effort=0 velocity=0
- added joint S1j: type revolute, parent S0, child S1, origin xyz=0.000000000 0.000000000 0.000000000 rpy=-1.5708     -1.5708     0.000000000, axis 0 0 1, limit lower=0 upper=0 effort=0 velocity=0
- added joint S2j: type revolute, parent S1, child S2, origin xyz= 0.3          0.000000000  0.000000000 rpy= 0.000000000  0.000000000  0.000000000, axis 0 0 1, limit lower=0 upper=0 effort=0 velocity=0
- added joint S3j: type revolute, parent S2, child S3, origin xyz= 0.3          0.000000000  -0.004      rpy= 0.000000000  0.000000000  1.5708    , axis 0 0 1, limit lower=0 upper=0 effort=0 velocity=0
- added joint S4j: type revolute, parent S3, child S4, origin xyz= 0.000000000  -0.1844      0.000000000 rpy= 1.5708      0.000000000  0.000000000, axis 0 0 1, limit lower=0 upper=0 effort=0 velocity=0
- joint J0_l: origin xyz=0 0 0 rpy=0 0 0 -> xyz=-0.008 0 0.3299 rpy=0 0 0; parent s4 -> S4
- joint J0_r: origin xyz=0 0 0 rpy=0 0 0 -> xyz=-0.008 0 0.3299 rpy=0 0 0; parent s4 -> S4
- joint arm_J1_l: origin xyz=0.000000000 0.209       0.000000000 rpy=-1.57079632 0.000000000 0.000000000 -> xyz=0.000000000 0.211       0.000000000 rpy=-1.57079632 0.000000000 0.000000000
- joint arm_J1_r: origin xyz=0.000000000 -0.209      0.000000000 rpy=-1.57079632 0.000000000 0.000000000 -> xyz=0.000000000 -0.211      0.000000000 rpy=-1.57079632 0.000000000 0.000000000
- joint arm_J3_l: origin xyz= 0.000000000  -0.310       0.000000000 rpy= 1.57079632   0.000000000  0.000000000 -> xyz= 0.000000000  -0.34955     0.000000000 rpy= 1.57079632   0.000000000  0.000000000
- joint arm_J3_r: origin xyz= 0.000000000  -0.310       0.000000000 rpy= -1.57079632  0.000000000  0.000000000 -> xyz= 0.000000000  -0.34955     0.000000000 rpy= -1.57079632  0.000000000  0.000000000
- joint arm_J4_l: origin xyz= 0.039        0.000000000  0.000000000 rpy= -1.57079632  0.000000000  0.000000000 -> xyz= 0.038567     0.000000000  0.000000000 rpy= -1.57079632  0.000000000  0.000000000
- joint arm_J4_r: origin xyz= 0.039        0.000000000  0.000000000 rpy= 1.57079632  0.000000000  0.000000000 -> xyz= 0.038567     0.000000000  0.000000000 rpy= 1.57079632  0.000000000  0.000000000
- joint arm_J5_l: origin xyz= 0.000000000  -0.310       0.000000000 rpy= 1.57079632  0.000000000  0.000000000 -> xyz= 0.000000000  -0.352       0.000000000 rpy= 1.57079632  0.000000000  0.000000000
- joint arm_J5_r: origin xyz= 0.000000000  -0.310       0.000000000 rpy= -1.57079632   0.000000000  0.000000000 -> xyz= 0.000000000  -0.352       0.000000000 rpy= -1.57079632   0.000000000  0.000000000
- joint arm_J6_l: origin xyz= 0.000000000  0.000000000  0.000000000 rpy= -1.57079632  -1.57079632  0.000000000 -> xyz= 0.000000000  0.000000000  0.000000000 rpy= -1.57079632  0.000000000  0.000000000
- joint arm_J6_r: origin xyz= 0.000000000  0.000000000  0.000000000 rpy= 1.57079632   1.57079632   0.000000000 -> xyz= 0.000000000  0.000000000  0.000000000 rpy= 1.57079632   0.000000000  0.000000000
- joint arm_J7_l: limit lower=-1.22173 upper=1.22173 effort=100 velocity=5.0 -> lower=-6.28319 upper=6.28319 effort=100 velocity=5.0; origin xyz= 0.067        0.000000000  0.000000000 rpy= 1.57079632   0.000000000  0.000000000 -> xyz= 0.000000000  -0.11  0.000000000 rpy= 1.57079632   0.000000000  0.000000000
- joint arm_J7_r: limit lower=-1.22173 upper=1.22173 effort=100 velocity=5.0 -> lower=-6.28319 upper=6.28319 effort=100 velocity=5.0; origin xyz= 0.067        0.000000000  0.000000000 rpy= -1.57079632  0.000000000  0.000000000 -> xyz= 0.000000000  -0.11  0.000000000 rpy= -1.57079632  0.000000000  0.000000000
- joint arm_J8_l: origin xyz=0.045 0 0 rpy=0 0 0 -> xyz=0 0 0 rpy=0 0 0
- joint arm_J8_r: origin xyz=0.045 0 0 rpy=0 0 0 -> xyz=0 0 0 rpy=0 0 0
- joint w0: child DP -> S0; origin xyz=0.0 0.0 0.0 rpy=0.0 0.0 3.14159 -> xyz=0.0 0.0 0.3040 rpy=0.0 0.0 0.0
